Commit message: updated car models and mpc code

File: car/urdf/simple_car.urdf (robot description, URDF)
Before this commit: robot simple_car, 10 links, 9 joints
Links:
- removed link trailer_load
- removed link wheel_rl
- removed link wheel_rr
- link hitch_link: mass None -> 5; geometry collision cylinder length=0.4 radius=0.05; visual cylinder length=0.4 radius=0.05
- link trailer_wheel_l: mass None -> 5; geometry collision cylinder length=0.1 radius=0.25; visual cylinder length=0.1 radius=0.25
- link trailer_wheel_r: mass None -> 5; geometry collision cylinder length=0.1 radius=0.25; visual cylinder length=0.1 radius=0.25
- link wheel_fl: mass None -> 5; geometry collision cylinder length=0.1 radius=0.25; visual cylinder length=0.1 radius=0.25
- link wheel_fr: mass None -> 5; geometry collision cylinder length=0.1 radius=0.25; visual cylinder length=0.1 radius=0.25
Joints:
- removed joint hitch_connect
- removed joint trailer_load_fixed
- removed joint wheel_rl_joint
- removed joint wheel_rr_joint
- added joint hitch_fixed: type fixed, parent base_link, child hitch_link, origin xyz=-1.6 0 0.2
- joint trailer_hinge: limit lower=-1.0 upper=1.0 -> lower=-1.2 upper=1.2; origin xyz=-0.6 0 0 -> xyz=0 0 0
- joint trailer_wheel_l_joint: axis (none) -> 0 1 0; limit (none) -> effort=0 velocity=100; origin xyz=-0.9 0.8 0.0 -> xyz=-1.8 0.7 0; type fixed -> revolute
- joint trailer_wheel_r_joint: axis (none) -> 0 1 0; limit (none) -> effort=0 velocity=100; origin xyz=-0.9 -0.8 0.0 -> xyz=-1.8 -0.7 0; type fixed -> revolute
